File: Hardware/backplane/backplane.kicad_pcb (KiCad board)
At the start: 2 copper layers, 132.1 x 109.2 mm, 27 parts, among them J1 Conn_02x08_Odd_Even, J10 345-050-520-202, J11 Conn_02x08_Odd_Even, J12 Screw_Terminal_01x04, J2 Conn_02x08_Odd_Even, J3 Conn_02x04_Odd_Even, J4 Conn_02x08_Odd_Even, J5 Conn_02x08_Odd_Even, J6 Conn_02x04_Odd_Even, J7 345-050-520-202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

Commit message: Fix backplane LEDs
Resolves issue #4
Parts:
- moved R3 7.62 mm to (153.7, 127.0), turned to 180 degrees
Connections:
- D2 pad 1: Net-(D2-Pad1) -> GND
- D3 pad 1: /-12V -> Net-(D3-Pad1)
- D3 pad 2: Net-(D2-Pad1) -> GND
- R3 pad 1: Net-(D2-Pad1) -> Net-(D3-Pad1)
- R3 pad 2: GND -> /-12V
Routing:
- net Net-(D2-Pad1): track 25.5 -> 0.00 mm
- net /-12V: track 253.8 -> 247.6 mm
- net Net-(D3-Pad1): track 0.00 -> 3.81 mm

Commit message: Change address decode on backplane
Resolves issue #3
Connections:
- U1 pad 1: /A12 -> /A11
- U1 pad 2: /A13 -> /A12
- U1 pad 3: /A14 -> /A13
- U1 pad 5: GND -> /A14
Routing:
- net /A11: track 133.1 -> 191.9 mm
- net /A14: track 181.4 -> 176.3 mm
- net /A13: track 183.7 -> 181.2 mm
- net /A12: track 192.2 -> 189.6 mm
Changed lines of the file:
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@@
     (thickness 1.6)
     (drawings 41)
-    (tracks 1087)
+    (tracks 1093)
     (zones 0)
     (modules 27)
@@
       (net 42 /~IOSEL2))
     (pad 5 thru_hole oval (at 0 10.16 180) (size 2.4 1.6) (drill 0.8) (layers *.Cu *.Mask)
-      (net 1 GND))
+      (net 20 /A14))
     (pad 12 thru_hole oval (at 7.62 10.16 180) (size 2.4 1.6) (drill 0.8) (layers *.Cu *.Mask)
       (net 43 /~IOSEL3))
@@
       (net 44 /~IOSEL4))
     (pad 3 thru_hole oval (at 0 5.08 180) (size 2.4 1.6) (drill 0.8) (layers *.Cu *.Mask)
-      (net 20 /A14))
+      (net 13 /A13))
     (pad 10 thru_hole oval (at 7.62 15.24 180) (size 2.4 1.6) (drill 0.8) (layers *.Cu *.Mask)
       (net 45 /~IOSEL5))
     (pad 2 thru_hole oval (at 0 2.54 180) (size 2.4 1.6) (drill 0.8) (layers *.Cu *.Mask)
-      (net 13 /A13))
+      (net 21 /A12))
     (pad 9 thru_hole oval (at 7.62 17.78 180) (size 2.4 1.6) (drill 0.8) (layers *.Cu *.Mask)
       (net 46 /~IOSEL6))
     (pad 1 thru_hole rect (at 0 0 180) (size 2.4 1.6) (drill 0.8) (layers *.Cu *.Mask)
-      (net 21 /A12))
+      (net 14 /A11))
     (model ${KISYS3DMOD}/Package_DIP.3dshapes/DIP-16_W7.62mm.wrl
       (at (xyz 0 0 0))
@@
   (segment (start 130.81 82.55) (end 129.54 83.82) (width 0.25) (layer F.Cu) (net 12))
   (segment (start 129.54 83.82) (end 127 83.82) (width 0.25) (layer F.Cu) (net 12) (status 20))
-  (segment (start 225.425 122.555) (end 223.52 124.46) (width 0.25) (layer B.Cu) (net 12) (status 20))
-  (segment (start 225.425 89.535) (end 225.425 122.555) (width 0.25) (layer B.Cu) (net 12))
-  (segment (start 224.79 88.9) (end 225.425 89.535) (width 0.25) (layer B.Cu) (net 12))
-  (segment (start 223.52 88.9) (end 224.79 88.9) (width 0.25) (layer B.Cu) (net 12) (status 10))
   (segment (start 212.09 83.82) (end 203.2 83.82) (width 0.25) (layer F.Cu) (net 12) (status 20))
   (segment (start 218.44 90.17) (end 212.09 83.82) (width 0.25) (layer F.Cu) (net 12))
@@
   (segment (start 123.19 82.55) (end 113.03 82.55) (width 0.25) (layer F.Cu) (net 12))
   (segment (start 127 83.82) (end 124.46 83.82) (width 0.25) (layer F.Cu) (net 12) (status 10))
+  (segment (start 225.425 122.555) (end 223.52 124.46) (width 0.25) (layer B.Cu) (net 12))
+  (segment (start 223.52 88.9) (end 224.79 88.9) (width 0.25) (layer B.Cu) (net 12))
+  (segment (start 225.425 89.535) (end 225.425 122.555) (width 0.25) (layer B.Cu) (net 12))
+  (segment (start 224.79 88.9) (end 225.425 89.535) (width 0.25) (layer B.Cu) (net 12))
   (segment (start 203.2 78.74) (end 200.66 78.74) (width 0.25) (layer F.Cu) (net 13) (status 10))
   (segment (start 200.66 78.74) (end 199.39 77.47) (width 0.25) (layer F.Cu) (net 13))
@@
   (segment (start 130.81 77.47) (end 129.54 78.74) (width 0.25) (layer F.Cu) (net 13))
   (segment (start 129.54 78.74) (end 127 78.74) (width 0.25) (layer F.Cu) (net 13) (status 20))
-  (segment (start 225.425 134.62) (end 223.52 134.62) (width 0.25) (layer B.Cu) (net 13) (status 20))
-  (segment (start 226.695 133.35) (end 225.425 134.62) (width 0.25) (layer B.Cu) (net 13))
-  (segment (start 226.695 88.264295) (end 226.695 133.35) (width 0.25) (layer B.Cu) (net 13))
-  (segment (start 224.790705 86.36) (end 226.695 88.264295) (width 0.25) (layer B.Cu) (net 13))
-  (segment (start 223.52 86.36) (end 224.790705 86.36) (width 0.25) (layer B.Cu) (net 13) (status 10))
   (segment (start 209.55 78.74) (end 203.2 78.74) (width 0.25) (layer F.Cu) (net 13) (status 20))
   (segment (start 218.44 87.63) (end 209.55 78.74) (width 0.25) (layer F.Cu) (net 13))
@@
   (segment (start 115.57 77.47) (end 106.68 86.36) (width 0.25) (layer F.Cu) (net 13))
   (segment (start 127 78.74) (end 124.46 78.74) (width 0.25) (layer F.Cu) (net 13) (status 10))
+  (segment (start 226.695 88.264295) (end 226.695 128.905) (width 0.25) (layer B.Cu) (net 13))
+  (segment (start 226.695 130.81) (end 226.695 128.905) (width 0.25) (layer B.Cu) (net 13))
+  (segment (start 224.790705 86.36) (end 226.695 88.264295) (width 0.25) (layer B.Cu) (net 13))
+  (segment (start 223.52 86.36) (end 224.790705 86.36) (width 0.25) (layer B.Cu) (net 13) (status 10))
+  (segment (start 225.425 132.08) (end 226.695 130.81) (width 0.25) (layer B.Cu) (net 13))
+  (segment (start 223.52 132.08) (end 225.425 132.08) (width 0.25) (layer B.Cu) (net 13))
   (segment (start 203.2 73.66) (end 200.66 73.66) (width 0.25) (layer F.Cu) (net 14) (status 10))
   (segment (start 200.66 73.66) (end 199.39 72.39) (width 0.25) (layer F.Cu) (net 14))
@@
   (segment (start 124.46 73.66) (end 123.19 72.39) (width 0.25) (layer F.Cu) (net 14))
   (segment (start 127 73.66) (end 124.46 73.66) (width 0.25) (layer F.Cu) (net 14) (status 10))
+  (segment (start 223.52 137.16) (end 225.425 137.16) (width 0.25) (layer B.Cu) (net 14))
+  (segment (start 224.79 83.82) (end 223.52 83.82) (width 0.25) (layer B.Cu) (net 14))
+  (segment (start 227.965 134.62) (end 227.965 86.995) (width 0.25) (layer B.Cu) (net 14))
+  (segment (start 227.965 86.995) (end 224.79 83.82) (width 0.25) (layer B.Cu) (net 14))
+  (segment (start 225.425 137.16) (end 227.965 134.62) (width 0.25) (layer B.Cu) (net 14))
   (segment (start 203.2 68.58) (end 200.66 68.58) (width 0.25) (layer F.Cu) (net 15) (status 10))
   (segment (start 200.66 68.58) (end 199.39 67.31) (width 0.25) (layer F.Cu) (net 15))
@@
   (segment (start 199.39 80.01) (end 200.66 81.28) (width 0.25) (layer F.Cu) (net 20))
   (segment (start 200.66 81.28) (end 203.2 81.28) (width 0.25) (layer F.Cu) (net 20) (status 20))
-  (segment (start 222.25 87.63) (end 220.98 88.9) (width 0.25) (layer B.Cu) (net 20) (status 20))
-  (segment (start 224.79 87.63) (end 222.25 87.63) (width 0.25) (layer B.Cu) (net 20))
-  (segment (start 226.06 88.9) (end 224.79 87.63) (width 0.25) (layer B.Cu) (net 20))
-  (segment (start 226.06 131.445) (end 226.06 88.9) (width 0.25) (layer B.Cu) (net 20))
-  (segment (start 225.425 132.08) (end 226.06 131.445) (width 0.25) (layer B.Cu) (net 20))
-  (segment (start 223.52 132.08) (end 225.425 132.08) (width 0.25) (layer B.Cu) (net 20) (status 10))
   (segment (start 210.82 81.28) (end 203.2 81.28) (width 0.25) (layer F.Cu) (net 20) (status 20))
   (segment (start 218.44 88.9) (end 210.82 81.28) (width 0.25) (layer F.Cu) (net 20))
@@
   (segment (start 102.87 87.63) (end 106.68 87.63) (width 0.25) (layer F.Cu) (net 20))
   (segment (start 101.6 88.9) (end 102.87 87.63) (width 0.25) (layer F.Cu) (net 20) (status 10))
+  (segment (start 222.25 87.63) (end 220.98 88.9) (width 0.25) (layer B.Cu) (net 20))
+  (segment (start 224.79 87.63) (end 222.25 87.63) (width 0.25) (layer B.Cu) (net 20))
+  (segment (start 223.52 127) (end 225.425 127) (width 0.25) (layer B.Cu) (net 20))
+  (segment (start 226.06 126.365) (end 226.06 88.9) (width 0.25) (layer B.Cu) (net 20))
+  (segment (start 225.425 127) (end 226.06 126.365) (width 0.25) (layer B.Cu) (net 20))
+  (segment (start 226.06 88.9) (end 224.79 87.63) (width 0.25) (layer B.Cu) (net 20))
   (segment (start 127 76.2) (end 129.54 76.2) (width 0.25) (layer F.Cu) (net 21) (status 10))
   (segment (start 129.54 76.2) (end 130.81 74.93) (width 0.25) (layer F.Cu) (net 21))
@@
   (segment (start 180.34 76.2) (end 181.61 74.93) (width 0.25) (layer F.Cu) (net 21))
   (segment (start 177.8 76.2) (end 180.34 76.2) (width 0.25) (layer F.Cu) (net 21) (status 10))
-  (segment (start 222.25 85.09) (end 220.98 86.36) (width 0.25) (layer B.Cu) (net 21) (status 20))
-  (segment (start 224.79 85.09) (end 222.25 85.09) (width 0.25) (layer B.Cu) (net 21))
-  (segment (start 227.33 87.63) (end 224.79 85.09) (width 0.25) (layer B.Cu) (net 21))
-  (segment (start 227.33 135.255) (end 227.33 87.63) (width 0.25) (layer B.Cu) (net 21))
-  (segment (start 225.425 137.16) (end 227.33 135.255) (width 0.25) (layer B.Cu) (net 21))
-  (segment (start 223.52 137.16) (end 225.425 137.16) (width 0.25) (layer B.Cu) (net 21) (status 10))
   (segment (start 208.28 76.2) (end 203.2 76.2) (width 0.25) (layer F.Cu) (net 21) (status 20))
   (segment (start 218.44 86.36) (end 208.28 76.2) (width 0.25) (layer F.Cu) (net 21))
@@
   (segment (start 123.19 74.93) (end 124.46 76.2) (width 0.25) (layer F.Cu) (net 21))
   (segment (start 101.6 86.36) (end 102.87 85.09) (width 0.25) (layer F.Cu) (net 21) (status 10))
+  (segment (start 222.25 85.09) (end 220.98 86.36) (width 0.25) (layer B.Cu) (net 21) (status 20))
+  (segment (start 227.33 132.715) (end 227.33 87.63) (width 0.25) (layer B.Cu) (net 21))
+  (segment (start 223.52 134.62) (end 225.425 134.62) (width 0.25) (layer B.Cu) (net 21))
+  (segment (start 225.425 134.62) (end 227.33 132.715) (width 0.25) (layer B.Cu) (net 21))
+  (segment (start 227.33 87.63) (end 224.79 85.09) (width 0.25) (layer B.Cu) (net 21))
+  (segment (start 224.79 85.09) (end 222.25 85.09) (width 0.25) (layer B.Cu) (net 21))
   (segment (start 127 71.12) (end 129.54 71.12) (width 0.25) (layer F.Cu) (net 22) (status 10))
   (segment (start 129.54 71.12) (end 130.81 69.85) (width 0.25) (layer F.Cu) (net 22))

Commit message: Increment backplane rev & date
Other:
- board text added: "Rev 2 20211224 rjh"
- board text removed: "Rev 1 20211206 rjh"
Changed lines of the file:
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@@
   (title_block
     (title "Compe 6502 Prototyping Backplane")
-    (date 2021-12-06)
-    (rev 1)
+    (date 2021-12-24)
+    (rev 2)
     (company rjh)
     (comment 1 "CC-BY-SA 4.0")
@@
     )
   )
-  (gr_text "Rev 1\n20211206 rjh" (at 184.15 138.43) (layer B.SilkS)
+  (gr_text "Rev 2\n20211224 rjh" (at 184.15 138.43) (layer B.SilkS)
     (effects (font (size 1 1) (thickness 0.15)) (justify mirror))
   )
@@
     (effects (font (size 1.5 1.5) (thickness 0.25)))
   )
-  (gr_text "Rev 1\n20211206 rjh" (at 184.15 138.43) (layer F.SilkS)
+  (gr_text "Rev 2\n20211224 rjh" (at 184.15 138.43) (layer F.SilkS)
     (effects (font (size 1 1) (thickness 0.15)))
   )
