File: Hardware/backplane/backplane.sch (KiCad schematic (older format))
At the start: 27 parts, among them J1 Conn_02x08_Odd_Even, J10 345-050-520-202, J11 Conn_02x08_Odd_Even, J12 Screw_Terminal_01x04, J2 Conn_02x08_Odd_Even, J3 Conn_02x04_Odd_Even, J4 Conn_02x08_Odd_Even, J5 Conn_02x08_Odd_Even, J6 Conn_02x04_Odd_Even, J7 345-050-520-202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

Commit message: Fix backplane LEDs
Resolves issue #4
Connections:
- net -12V: now also R3.2; no longer D3.1 (K)
- net GND: now also D2.1 (K), D3.2 (A); no longer R3.2
- new net: D3.1 (K), R3.1
Other:
- moved on the sheet: R3
Changed lines of the file:
@@
 Text Label 8550 1850 2    50   ~ 0
 A15
-Text Label 8550 1550 2    50   ~ 0
-A14
 Text Label 8550 1450 2    50   ~ 0
 A13
@@
 	8600 1950 8550 1950
 Wire Wire Line
-	8550 1950 8550 2050
-Wire Wire Line
 	8550 2050 8600 2050
-Connection ~ 8550 2050
 Wire Wire Line
 	8550 2050 8550 2100
@@
 L Device:R_Small R3
 U 1 1 625A4393
-P 8900 4350
-F 0 "R3" V 8704 4350 50  0000 C CNN
-F 1 "3K3" V 8795 4350 50  0000 C CNN
-F 2 "Resistor_THT:R_Axial_DIN0207_L6.3mm_D2.5mm_P7.62mm_Horizontal" H 8900 4350 50  0001 C CNN
-F 3 "~" H 8900 4350 50  0001 C CNN
-F 4 "CF14JT3K30" H 8900 4350 50  0001 C CNN "MPN"
-F 5 "Stackpole" H 8900 4350 50  0001 C CNN "Manufacturer"
-	1    8900 4350
+P 8900 4750
+F 0 "R3" V 9004 4750 50  0000 C CNN
+F 1 "3K3" V 9095 4750 50  0000 C CNN
+F 2 "Resistor_THT:R_Axial_DIN0207_L6.3mm_D2.5mm_P7.62mm_Horizontal" H 8900 4750 50  0001 C CNN
+F 3 "~" H 8900 4750 50  0001 C CNN
+F 4 "CF14JT3K30" H 8900 4750 50  0001 C CNN "MPN"
+F 5 "Stackpole" H 8900 4750 50  0001 C CNN "Manufacturer"
+	1    8900 4750
 	0    1    1    0
 $EndComp
@@
 	3550 6600 3450 6600
 Wire Wire Line
-	8650 4350 8800 4350
-Wire Wire Line
-	9000 4350 9100 4350
-Wire Wire Line
-	8650 4750 9100 4750
+	8650 4750 8800 4750
+Wire Wire Line
+	9000 4750 9100 4750
+Wire Wire Line
+	8650 4350 9100 4350
+Text Label 8550 1550 2    50   ~ 0
+A14
+Connection ~ 8550 2050
+Wire Wire Line
+	8550 1950 8550 2050
 $EndSCHEMATC

Commit message: Change address decode on backplane
Resolves issue #3
Connections:
- net A11: now also U1.1 (A0)
- net A12: now also U1.2 (A1); no longer U1.1 (A0)
- net A13: now also U1.3 (A2); no longer U1.2 (A1)
- net A14: now also U1.5 (E2); no longer U1.3 (A2)
- net GND: no longer U1.5 (E2)
Changed lines of the file:
@@
 Text Label 8550 1850 2    50   ~ 0
 A15
+Text Label 8550 1550 2    50   ~ 0
+A13
 Text Label 8550 1450 2    50   ~ 0
-A13
-Text Label 8550 1350 2    50   ~ 0
 A12
 Wire Wire Line
@@
 Wire Wire Line
 	8650 4350 9100 4350
-Text Label 8550 1550 2    50   ~ 0
+Text Label 8550 1950 2    50   ~ 0
 A14
-Connection ~ 8550 2050
-Wire Wire Line
-	8550 1950 8550 2050
+Text Label 8550 1350 2    50   ~ 0
+A11
 $EndSCHEMATC
