File: Hardware/motherboard/AddressDecode.kicad_sch (KiCad schematic)
At the start: 7 parts, among them U10 74HC138, U11 74HC138, U12 74HC08, U13 74HC138, U14 74HC32, U5 74HC00, U9 74HC138

Commit message: Complete mobo first draft
Parts:
- added unit 1 of U9
- renumbered U9 to U1, U10 to U3, U14 to U4, U11 to U6, U5 to U7, U13 to U8, U12 to U9
Connections:
- net GND: now also U4.1, U4.2, U4.4, U4.5, U9.4, U9.5, U9.1, U9.2; no longer U4.10, U4.4, U4.5, U4.9, U9.12, U9.13
- net ~{C000-FFFF}: now also U4.9; no longer U4.1
- net ~{IOSEL6}: now also U9.11; no longer U9.3
- net ~{ROMEN}: now also U4.8; no longer U4.3
- net at U3.9 (O6): now also U9.12; no longer U9.1
- net at U3.7 (O7): now also U9.13; no longer U9.2
- net at U7.3: now also U4.10; no longer U4.2
- no-connect marks 15 -> 16

Commit message: Misc hardware work
Parts:
- added TP10, TP11, TP12, TP17, TP27, TP28, TP9: TestPoint, TestPoint:TestPoint_THTPad_D1.5mm_Drill0.7mm, symbol Connector:TestPoint
Connections:
- net ~{0000-3FFF}: now also TP9.1
- net ~{4000-7FFF}: now also TP10.1
- net ~{8000-BFFF}: now also TP11.1
- net ~{C000-FFFF}: now also TP12.1
- net ~{C000}: now also TP17.1
- net ~{RAMEN}: now also TP27.1
- net ~{ROMEN}: now also TP28.1
Other:
- moved on the sheet: U7C, U7D
