File: Hardware/motherboard/Expansion.kicad_sch (KiCad schematic)
At the start: 7 parts, among them J2 345-050-520-202, J3 345-050-520-202, J4 345-050-520-202, J5 345-050-520-202, J6 345-050-520-202, J7 345-050-520-202, J8 345-050-520-202

Commit message: Complete mobo first draft
Parts:
- renumbered J2 to J1, J8 to J10, J3 to J4, J4 to J5, J5 to J6, J6 to J8, J7 to J9
Changed lines of the file:
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@@
+    (stroke (width 0) (type default) (color 0 0 0 0))
+  )
+  (wire (pts (xy 106.68 114.3) (xy 106.68 115.57))
     (stroke (width 0) (type default) (color 0 0 0 0))
   )
@@
     (stroke (width 0) (type default) (color 0 0 0 0))
   )
-  (bus (pts (xy 247.65 140.97) (xy 190.5 140.97))
-    (stroke (width 0) (type default) (color 0 0 0 0))
-  )
   (wire (pts (xy 57.15 63.5) (xy 64.77 63.5))
     (stroke (width 0) (type default) (color 0 0 0 0))
@@
     (stroke (width 0) (type default) (color 0 0 0 0))
   )
+  (wire (pts (xy 106.68 109.22) (xy 106.68 110.49))
+    (stroke (width 0) (type default) (color 0 0 0 0))
+  )
   (wire (pts (xy 77.47 63.5) (xy 78.74 63.5))
     (stroke (width 0) (type default) (color 0 0 0 0))
@@
     (effects (font (size 1.27 1.27)) (justify right bottom))
   )
+  (label "+5V" (at 106.68 110.49 0)
+    (effects (font (size 1.27 1.27)) (justify left bottom))
+  )
   (label "PH2" (at 176.53 40.64 180)
     (effects (font (size 1.27 1.27)) (justify right bottom))
@@
   (label "GND" (at 92.71 45.72 180)
     (effects (font (size 1.27 1.27)) (justify right bottom))
+  )
+  (label "GND" (at 106.68 114.3 0)
+    (effects (font (size 1.27 1.27)) (justify left bottom))
   )
   (label "SYNC" (at 203.2 71.12 180)
@@
     (pin "1")
   )
+  (symbol (lib_id "power:+5V") (at 106.68 109.22 0) (unit 1)
+    (in_bom yes) (on_board yes) (fields_autoplaced)
+    (property "Reference" "#PWR0109" (id 0) (at 106.68 113.03 0)
+      (effects (font (size 1.27 1.27)) hide)
+    )
+    (property "Value" "+5V" (id 1) (at 106.68 105.6155 0))
+    (property "Footprint" "" (id 2) (at 106.68 109.22 0)
+      (effects (font (size 1.27 1.27)) hide)
+    )
+    (property "Datasheet" "" (id 3) (at 106.68 109.22 0)
+      (effects (font (size 1.27 1.27)) hide)
+    )
+    (pin "1")
+  )
   (symbol (lib_id "power:-12V") (at 114.3 115.57 180) (unit 1)
     (in_bom yes) (on_board yes) (fields_autoplaced)
@@
   (symbol (lib_id "Connector_Generic:Conn_02x25_Odd_Even") (at 72.39 60.96 0) (mirror y) (unit 1)
     (in_bom yes) (on_board yes)
-    (property "Reference" "J2" (id 0) (at 71.12 24.9682 0))
+    (property "Reference" "J1" (id 0) (at 71.12 24.9682 0))
     (property "Value" "345-050-520-202" (id 1) (at 71.12 27.2796 0))
     (property "Footprint" "footprints:EDAC_345-050-520-202" (id 2) (at 72.39 60.96 0)
@@
     (pin "9")
   )
+  (symbol (lib_id "power:GND") (at 106.68 115.57 0) (unit 1)
+    (in_bom yes) (on_board yes) (fields_autoplaced)
+    (property "Reference" "#PWR0110" (id 0) (at 106.68 121.92 0)
+      (effects (font (size 1.27 1.27)) hide)
+    )
+    (property "Value" "GND" (id 1) (at 106.68 120.1325 0))
+    (property "Footprint" "" (id 2) (at 106.68 115.57 0)
+      (effects (font (size 1.27 1.27)) hide)
+    )
+    (property "Datasheet" "" (id 3) (at 106.68 115.57 0)
+      (effects (font (size 1.27 1.27)) hide)
+    )
+    (pin "1")
+  )
   (symbol (lib_id "Connector_Generic:Conn_02x25_Odd_Even") (at 158.75 60.96 0) (mirror y) (unit 1)
     (in_bom yes) (on_board yes)
-    (property "Reference" "J5" (id 0) (at 157.48 24.9682 0))
+    (property "Reference" "J6" (id 0) (at 157.48 24.9682 0))
     (property "Value" "345-050-520-202" (id 1) (at 157.48 27.2796 0))
     (property "Footprint" "footprints:EDAC_345-050-520-202" (id 2) (at 158.75 60.96 0)
@@
   (symbol (lib_id "Connector_Generic:Conn_02x25_Odd_Even") (at 238.76 60.96 0) (mirror y) (unit 1)
     (in_bom yes) (on_board yes)
-    (property "Reference" "J8" (id 0) (at 237.49 24.9682 0))
+    (property "Reference" "J10" (id 0) (at 237.49 24.9682 0))
     (property "Value" "345-050-520-202" (id 1) (at 237.49 27.2796 0))
     (property "Footprint" "footprints:EDAC_345-050-520-202" (id 2) (at 238.76 60.96 0)
@@
   (symbol (lib_id "Connector_Generic:Conn_02x25_Odd_Even") (at 101.6 60.96 0) (mirror y) (unit 1)
     (in_bom yes) (on_board yes)
-    (property "Reference" "J3" (id 0) (at 100.33 24.9682 0))
+    (property "Reference" "J4" (id 0) (at 100.33 24.9682 0))
     (property "Value" "345-050-520-202" (id 1) (at 100.33 27.2796 0))
     (property "Footprint" "footprints:EDAC_345-050-520-202" (id 2) (at 101.6 60.96 0)
@@
   (symbol (lib_id "Connector_Generic:Conn_02x25_Odd_Even") (at 212.09 60.96 0) (mirror y) (unit 1)
     (in_bom yes) (on_board yes)
-    (property "Reference" "J7" (id 0) (at 210.82 24.9682 0))
+    (property "Reference" "J9" (id 0) (at 210.82 24.9682 0))
     (property "Value" "345-050-520-202" (id 1) (at 210.82 27.2796 0))
     (property "Footprint" "footprints:EDAC_345-050-520-202" (id 2) (at 212.09 60.96 0)
@@
   (symbol (lib_id "Connector_Generic:Conn_02x25_Odd_Even") (at 130.81 60.96 0) (mirror y) (unit 1)
     (in_bom yes) (on_board yes)
-    (property "Reference" "J4" (id 0) (at 129.54 24.9682 0))
+    (property "Reference" "J5" (id 0) (at 129.54 24.9682 0))
     (property "Value" "345-050-520-202" (id 1) (at 129.54 27.2796 0))
     (property "Footprint" "footprints:EDAC_345-050-520-202" (id 2) (at 130.81 60.96 0)
@@
   (symbol (lib_id "Connector_Generic:Conn_02x25_Odd_Even") (at 185.42 60.96 0) (mirror y) (unit 1)
     (in_bom yes) (on_board yes)
-    (property "Reference" "J6" (id 0) (at 184.15 24.9682 0))
+    (property "Reference" "J8" (id 0) (at 184.15 24.9682 0))
     (property "Value" "345-050-520-202" (id 1) (at 184.15 27.2796 0))
     (property "Footprint" "footprints:EDAC_345-050-520-202" (id 2) (at 185.42 60.96 0)

Commit message: Misc hardware work
Parts:
- added TP1, TP13, TP14, TP19, TP2, TP20, TP25, TP26, TP29, TP30, TP31, TP32, TP7, TP8: TestPoint, TestPoint:TestPoint_THTPad_D1.5mm_Drill0.7mm, symbol Connector:TestPoint
- renumbered J1 to J2
Connections:
- net ~{DEV0}: now also TP2.1
- net ~{DEV1}: now also TP8.1
- net ~{DEV2}: now also TP14.1
- net ~{DEV3}: now also TP20.1
- net ~{DEV4}: now also TP26.1
- net ~{DEV5}: now also TP30.1
- net ~{DEV6}: now also TP32.1
- net ~{IOSEL0}: now also TP1.1
- net ~{IOSEL1}: now also TP7.1
- net ~{IOSEL2}: now also TP13.1
- net ~{IOSEL3}: now also TP19.1
- net ~{IOSEL4}: now also TP25.1
- net ~{IOSEL5}: now also TP29.1
- net ~{IOSEL6}: now also TP31.1
Other:
- moved on the sheet: J10, J2, J4, J5, J6, J8, J9
