File: Hardware/motherboard/PowerDecoupling.kicad_sch (KiCad schematic)
At the start: 34 parts, among them J9 Conn_01x04

Commit message: Complete mobo first draft
Parts:
- added J3: Conn_01x02, Connector_PinHeader_2.54mm:PinHeader_1x02_P2.54mm_Vertical, symbol Connector_Generic:Conn_01x02
- added R4: 1K0, Resistor_SMD:R_0805_2012Metric, symbol Device:R_Small
- J2: renamed from J9; footprint (none) -> Connector_Molex:Molex_Micro-Fit_3.0_43045-0400_2x02_P3.00mm_Horizontal
- renumbered C22 to C10, C6 to C11, C11 to C12, C19 to C13, C18 to C14, C17 to C15, C15 to C16, C16 to C17, C13 to C18, C14 to C19, C4 to C2, C5 to C20, C23 to C21, C2 to C22, C3 to C23, C7 to C3, C20 to C4, C12 to C5, C21 to C6, C8 to C7, C9 to C8, C10 to C9, H3 to H2, H2 to H3, R6 to R1, R7 to R2, R8 to R3
Connections:
- net +5V: now also R4.2
- net -12V: now also C3.2, D3.1 (K); no longer C3.1, R3.1
- net GND: now also C3.1, R3.1, J3.2 (Pin_2); no longer C3.2, D3.2 (A)
- net at R3.2: now also D3.2 (A); no longer D3.1 (K)
- new net: J3.1 (Pin_1), R4.1
Other:
- moved on the sheet: D3

Commit message: Misc hardware work
Parts:
- added TP3, TP4, TP5, TP6: TestPoint, TestPoint:TestPoint_THTPad_D1.5mm_Drill0.7mm, symbol Connector:TestPoint
- renumbered J2 to J1
Connections:
- net +12V: now also TP5.1
- net +5V: now also TP6.1
- net -12V: now also TP3.1
- net GND: now also TP4.1
Other:
- moved on the sheet: C2, C3, D1, D2, D3, R1, R2, R3
