File: Hardware/motherboard/motherboard.kicad_pcb (KiCad board)
At the start: 2 copper layers, 167.6 x 134.6 mm, 61 parts, among them J1 Conn_01x02, J2 345-050-520-202, J3 345-050-520-202, J4 345-050-520-202, J5 345-050-520-202, J6 345-050-520-202, J7 345-050-520-202, J8 345-050-520-202, U1 74HC74, U10 74HC138, U11 74HC138, U12 74HC08, U13 74HC138, U14 74HC32, U2 74HC08, U3 DS1813, U4 74HC161, U5 74HC00, U6 W65C02SxxPL, U7 28C256, U8 62256, U9 74HC138, X1 14.31818MHz

Commit message: Complete mobo first draft
Parts:
- added J2: Conn_01x04, Connector_Molex:Molex_Micro-Fit_3.0_43045-0400_2x02_P3.00mm_Horizontal, F.Cu at (74.7, 147.3)
- added J3: Conn_01x02, Connector_PinHeader_2.54mm:PinHeader_1x02_P2.54mm_Vertical, F.Cu at (78.7, 154.9)
- added R4: 1K0, Resistor_SMD:R_0805_2012Metric, F.Cu at (78.7, 151.2)
- added SW1: SW_Push, Button_Switch_SMD:SW_SPST_B3S-1000, F.Cu at (166.6, 150.9)
- added kibuzzard-1: G***, kibuzzard-61E4A308, F.Cu at (70.4, 152.9)
- added kibuzzard-10: G***, kibuzzard-61E47B7F, F.Cu at (198.1, 110.7)
- added kibuzzard-11: G***, kibuzzard-61E4DE7F, F.Cu at (221.0, 147.3)
- added kibuzzard-12: G***, kibuzzard-61E47B85, F.Cu at (223.5, 110.7)
- added kibuzzard-13: G***, kibuzzard-61E4DE7F, B.Cu at (221.0, 147.3)
- added kibuzzard-2: G***, kibuzzard-61E47B61, F.Cu at (71.1, 110.7)
- added kibuzzard-3: G***, kibuzzard-61E48162, F.Cu at (78.7, 115.7)
- added kibuzzard-4: G***, kibuzzard-61E4816D, F.Cu at (78.7, 123.3)
- added kibuzzard-5: G***, kibuzzard-61E48181, F.Cu at (78.7, 130.9)
- added kibuzzard-6: G***, kibuzzard-61E47B68, F.Cu at (96.5, 110.7)
- added kibuzzard-7: G***, kibuzzard-61E47B6E, F.Cu at (121.9, 110.7)
- added kibuzzard-8: G***, kibuzzard-61E47B74, F.Cu at (147.3, 110.7)
- added kibuzzard-9: G***, kibuzzard-61E47B79, F.Cu at (172.7, 110.7)
- moved J7 13.8 mm to (160.8, 154.9), turned to -90 degrees
- moved C1 12.7 mm to (71.1, 120.0)
- moved C2 12.7 mm to (71.1, 127.6)
- moved D2 12.7 mm to (78.7, 125.1)
- moved D3 12.7 mm to (78.7, 132.7)
- moved R1 12.7 mm to (78.7, 120.0)
- moved R2 12.7 mm to (78.7, 127.6)
- moved C3 12.7 mm to (71.1, 135.3)
- moved D1 12.7 mm to (78.7, 117.5)
- moved R3 12.7 mm to (78.7, 135.3)
- moved C12 9.42 mm to (117.9, 113.4), turned to 90 degrees
- moved C23 7.85 mm to (188.9, 113.7), turned to 0 degrees
- moved C11 7.62 mm to (102.6, 142.1)
- moved U13 7.62 mm to (188.0, 132.1)
- moved U2 7.62 mm to (91.4, 132.1)
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- renumbered C22 to C10, C6 to C11, C11 to C12, C19 to C13, C18 to C14, C17 to C15, C15 to C16, C16 to C17, C13 to C18, C14 to C19, C4 to C2, C5 to C20, C23 to C21, C2 to C22, C3 to C23, C7 to C3, C20 to C4, C12 to C5, C21 to C6, C8 to C7, C9 to C8, C10 to C9, H3 to H2, H2 to H3, J2 to J1, J8 to J10, J3 to J4, J4 to J5, J5 to J6, J1 to J7, J6 to J8, J7 to J9, R6 to R1, R7 to R2, R8 to R3, R4 to R5, R5 to R6, R1 to R7, R2 to R8, R3 to R9, U9 to U1, U2 to U10, U3 to U11, U6 to U12, U7 to U13, U8 to U14, U1 to U2, U10 to U3, U14 to U4, U4 to U5, U11 to U6, U5 to U7, U13 to U8, U12 to U9
Connections:
- C3 pad 1: -12V -> GND
- C3 pad 2: GND -> -12V
- D3 pad 1: Net-(D3-Pad1) -> -12V
- D3 pad 2: GND -> Net-(D3-Pad2)
- J1 pad 14: /Expansion/GND -> GND
- J1 pad 20: /Expansion/GND -> GND
- J1 pad 26: /Expansion/GND -> GND
- J1 pad 32: /Expansion/GND -> GND
- J1 pad 33: /Expansion/GND -> GND
- J1 pad 38: /Expansion/GND -> GND
- J1 pad 46: /Expansion/GND -> GND
- J1 pad 6: /Expansion/+5V -> +5V
- J1 pad 8: /Expansion/GND -> GND
- J10 pad 14: /Expansion/GND -> GND
- J10 pad 20: /Expansion/GND -> GND
- J10 pad 26: /Expansion/GND -> GND
- J10 pad 32: /Expansion/GND -> GND
- J10 pad 33: /Expansion/GND -> GND
- J10 pad 38: /Expansion/GND -> GND
- J10 pad 46: /Expansion/GND -> GND
- J10 pad 6: /Expansion/+5V -> +5V
- J10 pad 8: /Expansion/GND -> GND
- J4 pad 14: /Expansion/GND -> GND
- J4 pad 20: /Expansion/GND -> GND
- J4 pad 26: /Expansion/GND -> GND
- J4 pad 32: /Expansion/GND -> GND
- J4 pad 33: /Expansion/GND -> GND
- J4 pad 38: /Expansion/GND -> GND
- J4 pad 46: /Expansion/GND -> GND
- J4 pad 6: /Expansion/+5V -> +5V
- J4 pad 8: /Expansion/GND -> GND
- J5 pad 14: /Expansion/GND -> GND
- J5 pad 20: /Expansion/GND -> GND
- J5 pad 26: /Expansion/GND -> GND
- J5 pad 32: /Expansion/GND -> GND
- J5 pad 33: /Expansion/GND -> GND
- J5 pad 38: /Expansion/GND -> GND
- J5 pad 46: /Expansion/GND -> GND
- J5 pad 6: /Expansion/+5V -> +5V
- J5 pad 8: /Expansion/GND -> GND
- J6 pad 14: /Expansion/GND -> GND
- J6 pad 20: /Expansion/GND -> GND
- J6 pad 26: /Expansion/GND -> GND
- J6 pad 32: /Expansion/GND -> GND
- J6 pad 33: /Expansion/GND -> GND
- J6 pad 38: /Expansion/GND -> GND
- J6 pad 46: /Expansion/GND -> GND
- J6 pad 6: /Expansion/+5V -> +5V
- J6 pad 8: /Expansion/GND -> GND
- J8 pad 14: /Expansion/GND -> GND
- J8 pad 20: /Expansion/GND -> GND
- J8 pad 26: /Expansion/GND -> GND
- J8 pad 32: /Expansion/GND -> GND
- J8 pad 33: /Expansion/GND -> GND
- J8 pad 38: /Expansion/GND -> GND
- J8 pad 46: /Expansion/GND -> GND
- J8 pad 6: /Expansion/+5V -> +5V
- J8 pad 8: /Expansion/GND -> GND
- J9 pad 14: /Expansion/GND -> GND
- J9 pad 20: /Expansion/GND -> GND
- J9 pad 26: /Expansion/GND -> GND
- J9 pad 32: /Expansion/GND -> GND
- J9 pad 33: /Expansion/GND -> GND
- J9 pad 38: /Expansion/GND -> GND
- J9 pad 46: /Expansion/GND -> GND
- J9 pad 6: /Expansion/+5V -> +5V
- J9 pad 8: /Expansion/GND -> GND
- R3 pad 1: -12V -> GND
- R3 pad 2: Net-(D3-Pad1) -> Net-(D3-Pad2)
- U3 pad 7: Net-(U10-Pad7) -> Net-(U3-Pad7)
- U3 pad 9: Net-(U10-Pad9) -> Net-(U3-Pad9)
- U4 pad 1: /AddressDecode/~{C000-FFFF} -> GND
- U4 pad 10: GND -> Net-(U4-Pad10)
- U4 pad 2: Net-(U14-Pad2) -> GND
- U4 pad 3: /~{ROMEN} -> unconnected-(U4-Pad3)
- U4 pad 8: unconnected-(U14-Pad8) -> /~{ROMEN}
- U4 pad 9: GND -> /AddressDecode/~{C000-FFFF}
- U7 pad 3: Net-(U14-Pad2) -> Net-(U4-Pad10)
- U9 pad 1: Net-(U10-Pad9) -> GND
- U9 pad 11: unconnected-(U12-Pad11) -> /~{IOSEL6}
- U9 pad 12: GND -> Net-(U3-Pad9)
- U9 pad 13: GND -> Net-(U3-Pad7)
- U9 pad 2: Net-(U10-Pad7) -> GND
- U9 pad 3: /~{IOSEL6} -> unconnected-(U9-Pad3)
- U9 pad 4: (no net) -> GND
- U9 pad 5: (no net) -> GND
- U9 pad 6: (no net) -> unconnected-(U9-Pad6)
Routing:
- net +5V: track 75.3 -> 825.9 mm, vias 0 -> 13
- net /A8: track 50.5 -> 359.3 mm, vias 1 -> 4
- net /A11: track 55.0 -> 358.8 mm, vias 2 -> 5
- net /A9: track 50.9 -> 350.0 mm, vias 1 -> 4
- net /A12: track 41.9 -> 339.2 mm, vias 1 -> 5
- net /A10: track 62.1 -> 357.3 mm, vias 1 -> 4
- net /A13: track 42.2 -> 328.8 mm, vias 2 -> 6
- net /A0: track 76.9 -> 362.9 mm, vias 1 -> 4
- net -12V: track 0.00 -> 281.9 mm, vias 0 -> 1
- net /A1: track 70.8 -> 351.5 mm, vias 1 -> 4
- net +12V: track 0.00 -> 277.0 mm, vias 0 -> 2
- net /A2: track 67.3 -> 341.4 mm, vias 1 -> 4
- net /R~{W}: track 0.00 -> 269.7 mm, vias 0 -> 1
- net /A3: track 67.4 -> 336.1 mm, vias 1 -> 4
- net /A14: track 41.6 -> 305.8 mm, vias 1 -> 4
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Other:
- board text added: "Mainboard rjh - rev ${REVISION} ${ISSUE_DATE}"
- board text added: "PWR LED"
- board text added: "RESET"

Commit message: Misc hardware work
Parts:
- added TP1: TestPoint, TestPoint:TestPoint_THTPad_D1.5mm_Drill0.7mm, F.Cu at (78.7, 82.5)
- added TP10: TestPoint, TestPoint:TestPoint_THTPad_D1.5mm_Drill0.7mm, F.Cu at (92.2, 110.5)
- added TP11: TestPoint, TestPoint:TestPoint_THTPad_D1.5mm_Drill0.7mm, F.Cu at (99.1, 118.7)
- added TP12: TestPoint, TestPoint:TestPoint_THTPad_D1.5mm_Drill0.7mm, F.Cu at (99.1, 121.3)
- added TP13: TestPoint, TestPoint:TestPoint_THTPad_D1.5mm_Drill0.7mm, F.Cu at (114.3, 83.8)
- added TP14: TestPoint, TestPoint:TestPoint_THTPad_D1.5mm_Drill0.7mm, F.Cu at (114.3, 86.4)
- added TP15: TestPoint, TestPoint:TestPoint_THTPad_D1.5mm_Drill0.7mm, F.Cu at (116.1, 152.3)
- added TP16: TestPoint, TestPoint:TestPoint_THTPad_D1.5mm_Drill0.7mm, F.Cu at (117.9, 133.6)
- added TP17: TestPoint, TestPoint:TestPoint_THTPad_D1.5mm_Drill0.7mm, F.Cu at (133.3, 116.8)
- added TP18: TestPoint, TestPoint:TestPoint_THTPad_D1.5mm_Drill0.7mm, F.Cu at (137.7, 152.4)
- added TP19: TestPoint, TestPoint:TestPoint_THTPad_D1.5mm_Drill0.7mm, F.Cu at (139.7, 83.8)
- added TP2: TestPoint, TestPoint:TestPoint_THTPad_D1.5mm_Drill0.7mm, F.Cu at (78.7, 85.1)
- added TP20: TestPoint, TestPoint:TestPoint_THTPad_D1.5mm_Drill0.7mm, F.Cu at (139.7, 86.4)
- added TP21: TestPoint, TestPoint:TestPoint_THTPad_D1.5mm_Drill0.7mm, F.Cu at (144.8, 152.9)
- added TP22: TestPoint, TestPoint:TestPoint_THTPad_D1.5mm_Drill0.7mm, F.Cu at (147.8, 146.3)
- added TP23: TestPoint, TestPoint:TestPoint_THTPad_D1.5mm_Drill0.7mm, F.Cu at (147.8, 148.8)
- added TP24: TestPoint, TestPoint:TestPoint_THTPad_D1.5mm_Drill0.7mm, F.Cu at (159.6, 112.0)
- added TP25: TestPoint, TestPoint:TestPoint_THTPad_D1.5mm_Drill0.7mm, F.Cu at (165.1, 83.8)
- added TP26: TestPoint, TestPoint:TestPoint_THTPad_D1.5mm_Drill0.7mm, F.Cu at (165.1, 86.4)
- added TP27: TestPoint, TestPoint:TestPoint_THTPad_D1.5mm_Drill0.7mm, F.Cu at (184.4, 144.1)
- added TP28: TestPoint, TestPoint:TestPoint_THTPad_D1.5mm_Drill0.7mm, F.Cu at (203.2, 113.8)
- added TP29: TestPoint, TestPoint:TestPoint_THTPad_D1.5mm_Drill0.7mm, F.Cu at (205.7, 82.5)
- added TP3: TestPoint, TestPoint:TestPoint_THTPad_D1.5mm_Drill0.7mm, F.Cu at (83.8, 138.4)
- added TP30: TestPoint, TestPoint:TestPoint_THTPad_D1.5mm_Drill0.7mm, F.Cu at (205.7, 85.1)
- added TP31: TestPoint, TestPoint:TestPoint_THTPad_D1.5mm_Drill0.7mm, F.Cu at (215.9, 83.8)
- added TP32: TestPoint, TestPoint:TestPoint_THTPad_D1.5mm_Drill0.7mm, F.Cu at (215.9, 86.4)
- added TP4: TestPoint, TestPoint:TestPoint_THTPad_D1.5mm_Drill0.7mm, F.Cu at (83.8, 141.6)
- added TP5: TestPoint, TestPoint:TestPoint_THTPad_D1.5mm_Drill0.7mm, F.Cu at (87.0, 138.4)
- added TP6: TestPoint, TestPoint:TestPoint_THTPad_D1.5mm_Drill0.7mm, F.Cu at (87.0, 141.6)
- added TP7: TestPoint, TestPoint:TestPoint_THTPad_D1.5mm_Drill0.7mm, F.Cu at (88.9, 83.8)
- added TP8: TestPoint, TestPoint:TestPoint_THTPad_D1.5mm_Drill0.7mm, F.Cu at (88.9, 86.4)
- added TP9: TestPoint, TestPoint:TestPoint_THTPad_D1.5mm_Drill0.7mm, F.Cu at (89.5, 110.5)
- moved kibuzzard-13 3.82 mm to (217.2, 147.3), turned to -90 degrees
- moved kibuzzard-11 3.81 mm to (217.2, 147.3), turned to 90 degrees
- moved J1 3.42 mm to (72.4, 144.8), turned to 180 degrees
- moved kibuzzard-2 2.59 mm to (70.9, 155.4)
- renumbered J2 to J1, J1 to J2, kibuzzard-2 to kibuzzard-1, kibuzzard-1 to kibuzzard-2
Routing:
- net +12V: track 277.0 -> 289.3 mm
- net /~{IOSEL5}: track 114.0 -> 124.7 mm
- net /~{IOSEL0}: track 65.2 -> 75.9 mm
- net /~{DEV5}: track 81.0 -> 91.7 mm
- net /~{DEV0}: track 96.1 -> 106.8 mm
- net /AddressDecode/~{C000-FFFF}: track 55.4 -> 63.1 mm
- net +5V: track 825.9 -> 832.1 mm
- net /~{IOSEL4}: track 89.1 -> 94.2 mm
- net /~{IOSEL3}: track 65.4 -> 70.5 mm
- net /~{DEV4}: track 54.0 -> 59.1 mm
- net /~{DEV3}: track 29.3 -> 34.4 mm
- net /~{IOSEL1}: track 41.4 -> 46.5 mm
- net /~{DEV2}: track 52.4 -> 57.5 mm
- net /~{IOSEL6}: track 122.5 -> 127.6 mm
- net /~{DEV6}: track 116.8 -> 121.8 mm
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