File: Hardware/motherboard/motherboard.kicad_sch (KiCad schematic)
At the start: 15 parts, among them J1 Conn_01x02, U1 74HC74, U2 74HC08, U3 DS1813, U4 74HC161, U5 74HC00, U6 W65C02SxxPL, U7 28C256, U8 62256, X1 14.31818MHz

Commit message: Complete mobo first draft
Parts:
- added SW1: SW_Push, Button_Switch_SMD:SW_SPST_B3S-1000, symbol Switch:SW_Push
- renumbered J1 to J7, R4 to R5, R5 to R6, R1 to R7, R2 to R8, R3 to R9, U2 to U10, U3 to U11, U6 to U12, U7 to U13, U8 to U14, U1 to U2, U4 to U5, U5 to U7
Connections:
- net GND: now also SW1.2
- net ~{RES}: now also SW1.1
Other:
- moved on the sheet: J7

Commit message: Misc hardware work
Parts:
- added TP15, TP16, TP18, TP21, TP22, TP23, TP24: TestPoint, TestPoint:TestPoint_THTPad_D1.5mm_Drill0.7mm, symbol Connector:TestPoint
Connections:
- net 14M: now also TP15.1
- net BE: now also TP21.1
- net BE_{CPU}: now also TP23.1
- net PH2: now also TP16.1
- net PH2_{CPU}: now also TP22.1
- net R~{W}: now also TP24.1
- net ~{DMA}: now also TP18.1
Other:
- moved on the sheet: U10B
